File: pcb/nRF52832_qfaa.sch (KiCad schematic (older format))
At the start: 39 parts, among them J1 Battery, J2 Conn_02x05_Odd_Even, J3 Conn_01x03_Male, U1 NRF52832, U2 LED-Button, U3 TLV75533PDBVR, U4 SPU0410HR5H, U5 W25Q32JVZP, X1 32MHz, X2 32.768kHz

Commit message: [pcb] added electrical OR for multiple power inputs
Parts:
- removed C17: 100nF, nRF52832_qfaa:RESC0402_N, symbol nRF52832_qfaa-eagle-import:CAPACITOR_0402_N
- removed R6: 330, Resistor_SMD:R_0402_1005Metric, symbol Device:R
- removed U4: SPU0410HR5H, voice_recorder:SPU0410HR5H, symbol custom:SPU0410HR5H
- added D? (x2): D_Schottky, symbol Device:D_Schottky
- added JP?: Jumper_2_Open, symbol Jumper:Jumper_2_Open
- added MK?: SPM1423HM4H, symbol Sensor_Audio:MP45DT02
- added R?: 1K, Resistor_SMD:R_0402_1005Metric, symbol Device:R
- added R?: 100, Resistor_SMD:R_0402_1005Metric, symbol Device:R
- added R? (x3): 100K, Resistor_SMD:R_0402_1005Metric, symbol Device:R
- R5: value 1M -> 100K
Connections:
- net labels added: BUTTON_LED, DBG_POWER_LATCH, LDO_SELF_LATCH, MCU_POWER_LATCH, PDM_CLK, PDM_DATA, VBAT_LEVEL
- net labels removed: MIC_OUT
- wire segments 187 -> 200
- no-connect marks 20 -> 16
Other:
- moved on the sheet: C10, C11, C13, C18, C19, C20, R2, R3, R4, R5, U3, X2

Commit message: hw version 1.1 draft
Parts:
- removed AE1: Antenna_Chip, voice_recorder:ANT_2450AT18B100, symbol Device:Antenna_Chip
- removed C18, C19: 10uF, Capacitor_SMD:C_0603_1608Metric, symbol nRF52832_qfaa-eagle-import:CAPACITOR_0402_N
- removed D? (x2): D_Schottky, symbol Device:D_Schottky
- removed J1: Battery, Connector_PinHeader_2.54mm:PinHeader_1x02_P2.54mm_Vertical, symbol Connector:Conn_01x02_Female
- removed J3: Conn_01x03_Male, Connector_PinHeader_2.54mm:PinHeader_1x03_P2.54mm_Vertical, symbol Connector:Conn_01x03_Male
- removed L2: 2.7nH, nRF52832_qfaa:RESC0402_N, symbol nRF52832_qfaa-eagle-import:INDUCTOR_0402_N
- removed R3, R4: 330, Resistor_SMD:R_0402_1005Metric, symbol Device:R
- removed R?: 1K, Resistor_SMD:R_0402_1005Metric, symbol Device:R
- removed R?: 100, Resistor_SMD:R_0402_1005Metric, symbol Device:R
- removed R? (x2): 100K, Resistor_SMD:R_0402_1005Metric, symbol Device:R
- removed U2: LED-Button, voice_recorder:LED_BUTTON, symbol custom:LED-Button
- removed U3: TLV75533PDBVR, Package_TO_SOT_SMD:SOT-23-5, symbol Regulator_Linear:TPS73133DBV
- added C22: DNP, Capacitor_SMD:C_0402_1005Metric, symbol nRF52832_qfaa-eagle-import:CAPACITOR_0402_N
- added H1, H2: MountingHole, nRF52832_qfaa:MountingHole_1mm, symbol Mechanical:MountingHole
- added S1: KMR221GLFS, SW_KMR221GLFS, symbol _button:KMR221GLFS
- added TP5: Antenna, TestPoint:TestPoint_Pad_D1.0mm, symbol Connector:TestPoint
- added TP6, TP7, TP8: TestPoint, TestPoint:TestPoint_Pad_D1.0mm, symbol Connector:TestPoint
- C10: renamed from C2; footprint nRF52832_qfaa:RESC0402_N -> Capacitor_SMD:C_0402_1005Metric
- C11, C12, C7: footprint nRF52832_qfaa:RESC0402_N -> Capacitor_SMD:C_0402_1005Metric
- C13: renamed from C1; footprint nRF52832_qfaa:RESC0402_N -> Capacitor_SMD:C_0402_1005Metric
- C14: renamed from C3; footprint nRF52832_qfaa:RESC0402_N -> Capacitor_SMD:C_0402_1005Metric
- C15: renamed from C20; footprint nRF52832_qfaa:RESC0402_N -> Capacitor_SMD:C_0402_1005Metric
- C16: renamed from C5; footprint nRF52832_qfaa:RESC0402_N -> Capacitor_SMD:C_0402_1005Metric
- C17: renamed from C15; footprint nRF52832_qfaa:RESC0402_N -> Capacitor_SMD:C_0402_1005Metric
- C18: renamed from C16; footprint nRF52832_qfaa:RESC0402_N -> Capacitor_SMD:C_0402_1005Metric
- C3: renamed from C13; footprint nRF52832_qfaa:RESC0402_N -> Capacitor_SMD:C_0402_1005Metric
- C4: renamed from C10; footprint nRF52832_qfaa:RESC0402_N -> Capacitor_SMD:C_0402_1005Metric
- C5: renamed from C9; footprint nRF52832_qfaa:RESC0603_N -> Capacitor_SMD:C_0402_1005Metric
- C6: renamed from C8; footprint nRF52832_qfaa:RESC0402_N -> Capacitor_SMD:C_0402_1005Metric
- C8: renamed from C6; footprint nRF52832_qfaa:RESC0402_N -> Capacitor_SMD:C_0402_1005Metric
- C9: renamed from C4; footprint nRF52832_qfaa:RESC0402_N -> Capacitor_SMD:C_0402_1005Metric
- D1: footprint LED_SMD:LED_Cree-PLCC4_2x2mm_CW -> nRF52832_qfaa:LED_Cree-PLCC4_2x2mm_CW
- JP1: renamed from JP?; footprint (none) -> Jumper:SolderJumper-2_P1.3mm_Open_RoundedPad1.0x1.5mm
- L2: renamed from L1; footprint nRF52832_qfaa:RESC0402_N -> Capacitor_SMD:C_0402_1005Metric
- MK1: renamed from MK?; footprint (none) -> Sensor_Audio:ST_HLGA-6_3.76x4.72mm_P1.65mm
- RN1: footprint Resistor_SMD:R_Array_Convex_4x0603 -> Resistor_SMD:R_Array_Convex_4x0402; LCSC C110021 -> C25726
- U2: renamed from U5; footprint Package_SON:WSON-8-1EP_6x5mm_P1.27mm_EP3.4x4.3mm -> nRF52832_qfaa:WSON-8-1EP_6x5mm_P1.27mm_EP3.4x4.3mm
- gave numbers to parts that had none: 1
- renumbered R5 to R1, R2 to R3, X2 to X1, X1 to X2
Connections:
- net labels added: MAIN_BUTTON, VSS
- net labels removed: +BATT, BUTTON, BUTTON_LED, LDO_EN, LDO_SELF_LATCH, P0.26
- wire segments 200 -> 155
- no-connect marks 16 -> 13
Other:
- moved on the sheet: C14, C15, C17, C18, C3, C5, C9, D1, J2, JP1, L2, MK1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

Commit message: [pcb] added fabrication outputs for the jlcpcb order
Parts:
- C10, C11, C12, C13: LCSC C2154389 -> C32949
- C14: LCSC C88902 -> C326068
- C15, C16, C18, C3, C6, C9: LCSC C541464 -> C1525
- C17: LCSC C92755 -> C52923
- C5: LCSC C109456 -> C77004
- D1: value ASMB-MTB0-0A3A2 -> ASMB-LTC2-0A335
- R1, R2: LCSC C93949 -> C25741
- R3: LCSC C168225 -> C25104
Changed lines of the file:
@@
 F 2 "Capacitor_SMD:C_0402_1005Metric" H 9300 2800 50  0001 C CNN
 F 3 "" H 9300 2800 50  0001 C CNN
-F 4 "C2154389" H 9300 2800 50  0001 C CNN "LCSC"
+F 4 "C32949" H 9300 2800 50  0001 C CNN "LCSC"
 	1    9300 2800
 	0    -1   -1   0
@@
 F 2 "Capacitor_SMD:C_0402_1005Metric" H 9300 3500 50  0001 C CNN
 F 3 "" H 9300 3500 50  0001 C CNN
-F 4 "C2154389" H 9300 3500 50  0001 C CNN "LCSC"
+F 4 "C32949" H 9300 3500 50  0001 C CNN "LCSC"
 	1    9300 3500
 	0    -1   -1   0
@@
 F 2 "Capacitor_SMD:C_0402_1005Metric" H 8400 4250 50  0001 C CNN
 F 3 "" H 8400 4250 50  0001 C CNN
-F 4 "C88902" H 8400 4250 50  0001 C CNN "LCSC"
+F 4 "C326068" H 8400 4250 50  0001 C CNN "LCSC"
 	1    8400 4250
 	-1   0    0    1
@@
 F 2 "Capacitor_SMD:C_0402_1005Metric" H 3650 2750 50  0001 C CNN
 F 3 "" H 3650 2750 50  0001 C CNN
-F 4 "C541464" H 3650 2750 50  0001 C CNN "LCSC"
+F 4 "C1525" H 3650 2750 50  0001 C CNN "LCSC"
 	1    3650 2750
 	1    0    0    -1
@@
 F 2 "Capacitor_SMD:C_0402_1005Metric" H 4400 5500 50  0001 C CNN
 F 3 "" H 4400 5500 50  0001 C CNN
-F 4 "C541464" H 4400 5500 50  0001 C CNN "LCSC"
+F 4 "C1525" H 4400 5500 50  0001 C CNN "LCSC"
 	1    4400 5500
 	1    0    0    -1
@@
 F 2 "Capacitor_SMD:C_0402_1005Metric" H 6600 2100 50  0001 C CNN
 F 3 "" H 6600 2100 50  0001 C CNN
-F 4 "C541464" H 6600 2100 50  0001 C CNN "LCSC"
+F 4 "C1525" H 6600 2100 50  0001 C CNN "LCSC"
 	1    6600 2100
 	1    0    0    -1
@@
 F 2 "Capacitor_SMD:C_0402_1005Metric" H 4650 2100 50  0001 C CNN
 F 3 "" H 4650 2100 50  0001 C CNN
-F 4 "C109456" H 4650 2100 50  0001 C CNN "LCSC"
+F 4 "C77004" H 4650 2100 50  0001 C CNN "LCSC"
 	1    4650 2100
 	1    0    0    -1
@@
 F 2 "Capacitor_SMD:C_0402_1005Metric" H 2000 3150 50  0001 C CNN
 F 3 "" H 2000 3150 50  0001 C CNN
-F 4 "C2154389" H 2000 3150 50  0001 C CNN "LCSC"
+F 4 "C32949" H 2000 3150 50  0001 C CNN "LCSC"
 	1    2000 3150
 	0    -1   -1   0
@@
 F 2 "Capacitor_SMD:C_0402_1005Metric" H 2000 3500 50  0001 C CNN
 F 3 "" H 2000 3500 50  0001 C CNN
-F 4 "C2154389" H 2000 3500 50  0001 C CNN "LCSC"
+F 4 "C32949" H 2000 3500 50  0001 C CNN "LCSC"
 	1    2000 3500
 	0    -1   -1   0
@@
 P 8400 6650
 F 0 "D1" H 8400 7167 50  0000 C CNN
-F 1 "ASMB-MTB0-0A3A2" H 8400 7076 50  0000 C CNN
+F 1 "ASMB-LTC2-0A335" H 8400 7076 50  0000 C CNN
 F 2 "nRF52832_qfaa:LED_Cree-PLCC4_2x2mm_CW" H 8400 7150 50  0001 C CNN
-F 3 "https://docs.broadcom.com/docs/AV02-4186EN" H 8400 6200 50  0001 C CNN
+F 3 "https://docs.broadcom.com/docs/ASMB-LTC2-0A335-DS" H 8400 6200 50  0001 C CNN
 	1    8400 6650
 	1    0    0    -1
@@
 F 2 "Capacitor_SMD:C_0402_1005Metric" H 1750 7150 50  0001 C CNN
 F 3 "" H 1750 7150 50  0001 C CNN
-F 4 "C92755" H 1750 7150 50  0001 C CNN "LCSC"
+F 4 "C52923" H 1750 7150 50  0001 C CNN "LCSC"
 	1    1750 7150
 	1    0    0    -1
@@
 F 2 "Capacitor_SMD:C_0402_1005Metric" H 2150 7150 50  0001 C CNN
 F 3 "" H 2150 7150 50  0001 C CNN
-F 4 "C541464" H 2150 7150 50  0001 C CNN "LCSC"
+F 4 "C1525" H 2150 7150 50  0001 C CNN "LCSC"
 	1    2150 7150
 	1    0    0    -1
@@
 F 2 "Resistor_SMD:R_0402_1005Metric" V 1030 4950 50  0001 C CNN
 F 3 "~" H 1100 4950 50  0001 C CNN
-F 4 "C168225" H 1100 4950 50  0001 C CNN "LCSC"
+F 4 "C25104" H 1100 4950 50  0001 C CNN "LCSC"
 	1    1100 4950
 	-1   0    0    1
@@
 F 2 "Resistor_SMD:R_0402_1005Metric" V 1930 2150 50  0001 C CNN
 F 3 "~" H 2000 2150 50  0001 C CNN
-F 4 "C93949" H 2000 2150 50  0001 C CNN "LCSC"
+F 4 "C25741" H 2000 2150 50  0001 C CNN "LCSC"
 	1    2000 2150
 	1    0    0    -1
@@
 F 2 "Capacitor_SMD:C_0402_1005Metric" H 950 5100 50  0001 C CNN
 F 3 "" H 950 5100 50  0001 C CNN
-F 4 "C541464" H 950 5100 50  0001 C CNN "LCSC"
+F 4 "C1525" H 950 5100 50  0001 C CNN "LCSC"
 	1    950  5100
 	0    1    1    0
@@
 F 2 "Resistor_SMD:R_0402_1005Metric" V 1780 1050 50  0001 C CNN
 F 3 "~" H 1850 1050 50  0001 C CNN
-F 4 "C93949" H 1850 1050 50  0001 C CNN "LCSC"
+F 4 "C25741" H 1850 1050 50  0001 C CNN "LCSC"
 	1    1850 1050
 	-1   0    0    -1
@@
 F 2 "Capacitor_SMD:C_0402_1005Metric" H 2150 1000 50  0001 C CNN
 F 3 "" H 2150 1000 50  0001 C CNN
-F 4 "C541464" H 2150 1000 50  0001 C CNN "LCSC"
+F 4 "C1525" H 2150 1000 50  0001 C CNN "LCSC"
 	1    2150 1000
 	1    0    0    -1
