File: pcb/power.sch (KiCad schematic (older format))
At the start: 21 parts, among them U3 TLV75533PDBVR, U4 BQ24078RGTR

Commit message: [pcb] added fabrication outputs for the jlcpcb order
Parts:
- C1, C2: LCSC C23733 -> C15525
- C19: LCSC C92755 -> C52923
- D3: LCSC (none) -> C72043
- R10, R11: LCSC C93949 -> C25741
- R4: LCSC C168225 -> C25744
- R5: LCSC C168225 -> C25867
- R6: LCSC (none) -> C67014
- R7: LCSC C93949 -> C25744
- R8: LCSC (none) -> C270651
- R9: LCSC C93949 -> C11702
- U4: LCSC (none) -> C15464
Changed lines of the file:
@@
 F 2 "Resistor_SMD:R_0402_1005Metric" V 6030 700 50  0001 C CNN
 F 3 "~" H 6100 700 50  0001 C CNN
-F 4 "C168225" H 6100 700 50  0001 C CNN "LCSC"
+F 4 "C25744" H 6100 700 50  0001 C CNN "LCSC"
 	1    6100 700
 	0    1    1    0
@@
 F 2 "Resistor_SMD:R_0402_1005Metric" V 6030 1100 50  0001 C CNN
 F 3 "~" H 6100 1100 50  0001 C CNN
-F 4 "C168225" H 6100 1100 50  0001 C CNN "LCSC"
+F 4 "C25867" H 6100 1100 50  0001 C CNN "LCSC"
 	1    6100 1100
 	0    1    1    0
@@
 F 2 "Resistor_SMD:R_0402_1005Metric" V 930 5100 50  0001 C CNN
 F 3 "~" H 1000 5100 50  0001 C CNN
-F 4 "C93949" H 1000 5100 50  0001 C CNN "LCSC"
+F 4 "C25741" H 1000 5100 50  0001 C CNN "LCSC"
 	1    1000 5100
 	1    0    0    -1
@@
 F 2 "Resistor_SMD:R_0402_1005Metric" V 930 5400 50  0001 C CNN
 F 3 "~" H 1000 5400 50  0001 C CNN
-F 4 "C93949" H 1000 5400 50  0001 C CNN "LCSC"
+F 4 "C25741" H 1000 5400 50  0001 C CNN "LCSC"
 	1    1000 5400
 	1    0    0    -1
@@
 F 2 "_other:VQFN-16-1EP_3x3mm_P0.5mm_EP1.45x1.45mm_ThermalVias" H 6450 3490 60  0001 C CNN
 F 3 "" H 5450 3250 60  0000 C CNN
+F 4 "C15464" H 5450 3250 50  0001 C CNN "LCSC"
 	1    5450 3250
 	1    0    0    -1
@@
 F 2 "Resistor_SMD:R_0402_1005Metric" V 5280 3000 50  0001 C CNN
 F 3 "~" H 5350 3000 50  0001 C CNN
-F 4 "C93949" H 5350 3000 50  0001 C CNN "LCSC"
+F 4 "C25744" H 5350 3000 50  0001 C CNN "LCSC"
 	1    5350 3000
 	1    0    0    -1
@@
 F 2 "Resistor_SMD:R_0402_1005Metric" V 7430 2950 50  0001 C CNN
 F 3 "~" H 7500 2950 50  0001 C CNN
-F 4 "" H 7500 2950 50  0001 C CNN "LCSC"
+F 4 "C67014" H 7500 2950 50  0001 C CNN "LCSC"
 	1    7500 2950
 	1    0    0    -1
@@
 F 2 "Resistor_SMD:R_0402_1005Metric" V 8330 4300 50  0001 C CNN
 F 3 "~" H 8400 4300 50  0001 C CNN
-F 4 "" H 8400 4300 50  0001 C CNN "LCSC"
+F 4 "C270651" H 8400 4300 50  0001 C CNN "LCSC"
 	1    8400 4300
 	1    0    0    -1
@@
 F 2 "Capacitor_SMD:C_0402_1005Metric" H 7850 3400 50  0001 C CNN
 F 3 "" H 7850 3400 50  0001 C CNN
-F 4 "C92755" H 7850 3400 50  0001 C CNN "LCSC"
+F 4 "C52923" H 7850 3400 50  0001 C CNN "LCSC"
 	1    7850 3400
 	1    0    0    -1
@@
 F 2 "Resistor_SMD:R_0402_1005Metric" V 7430 4600 50  0001 C CNN
 F 3 "~" H 7500 4600 50  0001 C CNN
-F 4 "C93949" H 7500 4600 50  0001 C CNN "LCSC"
+F 4 "C11702" H 7500 4600 50  0001 C CNN "LCSC"
 	1    7500 4600
 	1    0    0    1
@@
 F 2 "LED_SMD:LED_0603_1608Metric" H 7500 4300 50  0001 C CNN
 F 3 "~" H 7500 4300 50  0001 C CNN
+F 4 "C72043" H 7500 4300 50  0001 C CNN "LCSC"
 	1    7500 4300
 	0    1    1    0
@@
 F 2 "Capacitor_SMD:C_0402_1005Metric" H 8350 900 50  0001 C CNN
 F 3 "" H 8350 900 50  0001 C CNN
-F 4 "C23733" H 8350 900 50  0001 C CNN "LCSC"
+F 4 "C15525" H 8350 900 50  0001 C CNN "LCSC"
 	1    8350 900
 	1    0    0    -1
@@
 F 2 "Capacitor_SMD:C_0402_1005Metric" H 8750 900 50  0001 C CNN
 F 3 "" H 8750 900 50  0001 C CNN
-F 4 "C23733" H 8750 900 50  0001 C CNN "LCSC"
+F 4 "C15525" H 8750 900 50  0001 C CNN "LCSC"
 	1    8750 900
 	1    0    0    -1
