File: pcb/nRF52832_qfaa.kicad_sch (KiCad schematic)
At the start: 47 parts, among them J1 Conn_01x01_Female, J2 Conn_02x05_Odd_Even, U1 NRF52832, U2 W25Q32JVZP, X1 32.768kHz, X2 32MHz

Commit message: [pcb] finalizing layout of v1.3, only testpoints, teardrops and DRC is left
Parts:
- added C24: 1uF, Capacitor_SMD:C_0402_1005Metric, symbol nRF52832_qfaa-eagle-import:CAPACITOR_0402_N
- added C25: 100nF, Capacitor_SMD:C_0402_1005Metric, symbol nRF52832_qfaa-eagle-import:CAPACITOR_0402_N
- added R12: 33, Resistor_SMD:R_0402_1005Metric, symbol Device:R
- added R2, R4: 4.7k, Resistor_SMD:R_0402_1005Metric, symbol Device:R
- added U5: RV-4162-C7, _other:IC_RV-4162-C7, symbol RV-4162-C7:RV-4162-C7
Connections:
- net GND: now also C24.2, C25.2, U5.3 (VSS)
- net VCC: now also R2.1, R4.1
- net VSS: now also C24.1, C25.1, U5.5 (VDD)
- net FF_CLK: now reaches U1.38 (P0.26@38)
- net RTC_INT_N: now reaches U1.43 (P0.31@43)
- net RTC_INT_N: now also R12.1
- net P0.16 renamed I2C_SDA
- net I2C_SDA: now also R2.2, U5.1 (SDA)
- net P0.17 renamed I2C_SCL
- net I2C_SCL: now also R4.2, U5.8 (SCL)
- new net: U5.4 (NC), U5.7 (NC)
- new net: R12.2, U5.6 (~{INT})
- new net RTC_CLKOUT: U5.2 (CLKOUT)
- no-connect marks 14 -> 12
Other:
- moved on the sheet: H1, H2

Commit message: [pcb] finalized layout of v1.3
Parts:
- removed TP12, TP13, TP14, TP15, TP20, TP21, TP22, TP23: TestPoint, TestPoint:TestPoint_Pad_D1.0mm, symbol Connector:TestPoint
- added TP18, TP5: TestPoint, TestPoint:TestPoint_Pad_D1.0mm, symbol Connector:TestPoint
Connections:
- net I2C_SCL: now also TP5.1
- net I2C_SDA: now also TP18.1
