File: pcb/nRF52832_qfaa.kicad_sch (KiCad schematic)
At the start: 47 parts, among them J1 Conn_01x01_Female, J2 Conn_02x05_Odd_Even, U1 NRF52832, U2 W25Q32JVZP, X1 32.768kHz, X2 32MHz

Commit message: [pcb] version 1.3 (#75)
Changes:
    LDO voltage regulator replaced with DC-DC (expected increase in efficiency)
    added small-footprint RTC chip
    analog latch for regulator EN pin replaced with a digital flip-flop

Fixture:
    added Raspberry Pico to the PCB
    added current measurement setup
    planning to reduce hardware in use to a single PCB
Parts:
- removed TP12, TP13, TP14, TP15, TP20, TP21, TP22, TP23: TestPoint, TestPoint:TestPoint_Pad_D1.0mm, symbol Connector:TestPoint
- added C24: 1uF, Capacitor_SMD:C_0402_1005Metric, symbol nRF52832_qfaa-eagle-import:CAPACITOR_0402_N
- added C25: 100nF, Capacitor_SMD:C_0402_1005Metric, symbol nRF52832_qfaa-eagle-import:CAPACITOR_0402_N
- added R12: 33, Resistor_SMD:R_0402_1005Metric, symbol Device:R
- added R2, R4: 4.7k, Resistor_SMD:R_0402_1005Metric, symbol Device:R
- added TP18, TP5: TestPoint, TestPoint:TestPoint_Pad_D1.0mm, symbol Connector:TestPoint
- added U5: RV-4162-C7, _other:IC_RV-4162-C7, symbol RV-4162-C7:RV-4162-C7
Connections:
- net GND: now also C24.2, C25.2, U5.3 (VSS)
- net VCC: now also R2.1, R4.1
- net VSS: now also C24.1, C25.1, U5.5 (VDD)
- net FF_CLK: now reaches U1.38 (P0.26@38)
- net RTC_INT_N: now reaches U1.43 (P0.31@43)
- net RTC_INT_N: now also R12.1
- net P0.16 renamed I2C_SDA
- net I2C_SDA: now also R2.2, TP18.1, U5.1 (SDA)
- net P0.17 renamed I2C_SCL
- net I2C_SCL: now also R4.2, TP5.1, U5.8 (SCL)
- new net: U5.4 (NC), U5.7 (NC)
- new net: R12.2, U5.6 (~{INT})
- new net RTC_CLKOUT: U5.2 (CLKOUT)
- no-connect marks 14 -> 12
Other:
- moved on the sheet: H1, H2

Commit message: start laying out 1.4
Parts:
- removed C14: 0.8pF, Capacitor_SMD:C_0402_1005Metric, symbol nRF52832_qfaa-eagle-import:CAPACITOR_0402_N
- removed C16, C6, C9: 100nF, Capacitor_SMD:C_0402_1005Metric, symbol nRF52832_qfaa-eagle-import:CAPACITOR_0402_N
- removed C22: DNP, Capacitor_SMD:C_0402_1005Metric, symbol nRF52832_qfaa-eagle-import:CAPACITOR_0402_N
- removed C4: 1µF, Capacitor_SMD:C_0402_1005Metric, symbol nRF52832_qfaa-eagle-import:CAPACITOR_0603_N
- removed C5: 4.7µF, Capacitor_SMD:C_0402_1005Metric, symbol nRF52832_qfaa-eagle-import:CAPACITOR_0603_N
- removed C7: 100pF, Capacitor_SMD:C_0402_1005Metric, symbol nRF52832_qfaa-eagle-import:CAPACITOR_0402_N
- removed C8: N.M., Capacitor_SMD:C_0402_1005Metric, symbol nRF52832_qfaa-eagle-import:CAPACITOR_0402_N
- removed L2: 3.3nH, Capacitor_SMD:C_0402_1005Metric, symbol nRF52832_qfaa-eagle-import:INDUCTOR_0402_N
- removed TP11: TestPoint, TestPoint:TestPoint_Pad_D1.0mm, symbol Connector:TestPoint
- removed U1: NRF52832, nRF52832_qfaa:QFN40P600X600X90-48_N, symbol nRF52832_qfaa-eagle-import:NRF52832
- added C28, C29, C30, C31, C32, C33, C34, C35, C45: 100n, Capacitor_SMD:C_0201_0603Metric, symbol Device:C
- added C36: N.C, Capacitor_SMD:C_0201_0603Metric, symbol Device:C
- added C37, C38, C39, C40, C44: 1u, Capacitor_SMD:C_0402_1005Metric, symbol Device:C
- added C39(NP0)1: 100pF, Capacitor_SMD:C_0201_0603Metric, symbol Device:C
- added C41: 2.2u, Capacitor_SMD:C_0603_1608Metric, symbol Device:C
- added C42, C43: 4.7u, Capacitor_SMD:C_0603_1608Metric, symbol Device:C
- added C46: DNP, Capacitor_SMD:C_0201_0603Metric, symbol Device:C
- added C47: 0.7pF, Capacitor_SMD:C_0201_0603Metric, symbol Device:C
- added D2, D4: ASMB-LTC2-0A335, nRF52832_qfaa:LED_Cree-PLCC4_2x2mm_CW, symbol LED:ASMB-MTB0-0A3A2
- added J3: USB_B_Micro, Connector_USB:USB_Micro-B_Molex-105017-0001, symbol Connector:USB_B_Micro
- added L3, L4: 10uH, Inductor_SMD:L_0603_1608Metric, symbol Device:L
- added L5, L6: 15nH, Inductor_SMD:L_0201_0603Metric, symbol Device:L
- added L7: 2.2nH, Inductor_SMD:L_0201_0603Metric, symbol Device:L
- added R20: 4.7, Resistor_SMD:R_0201_0603Metric, symbol Device:R
- added RN2, RN3: R_Pack04, Resistor_SMD:R_Array_Convex_4x0402, symbol Device:R_Pack04
- added U7: NRF5340-QKAA-R7, _other:XCVR_NRF5340-QKAA-R7, symbol NRF5340:NRF5340-QKAA-R7
- C11, C12: footprint Capacitor_SMD:C_0402_1005Metric -> Capacitor_SMD:C_0201_0603Metric; LCSC C32949 -> (none)
- X1: footprint nRF52832_qfaa:XTAL_3215_N -> Crystal:Crystal_SMD_MicroCrystal_CM9V-T1A-2Pin_1.6x1.0mm; Digikey (none) -> https://www.digikey.de/de/products/detail/citizen-finedevic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
Connections:
- net GND: now also C28.2, C29.2, C30.2, C31.2, C32.2, C33.2, C34.2, C35.2, C36.2, C37.2, C38.2, C39(NP0)1.2, C39.2, C40.2, C41.1, C42.2, C43.2, C44.2, C45.2, C46.2, C47.2, U7.104 (VSS_PAD), U7.35 (VSS_PAD), U7.36 (VSS_PAD), U7.37 (VSS_PAD), U7.38 (VSS_PAD), U7.39 (VSS_PAD), U7.40 (VSS_PAD), U7.41 (VSS_PAD), U7.43 (VSS_PAD), U7.44 (VSS_PAD), U7.45 (VSS_PAD), U7.46 (VSS_PAD), U7.47 (VSS_PAD), U7.48 (VSS_PAD), U7.49 (VSS_PAD), U7.50 (VSS_PAD), U7.51 (VSS_PAD), U7.A25 (VSS), U7.B12 (VSS), U7.B26 (VSS), U7.G1 (VSS), U7.H2 (VSS), U7.J31 (VSS)
- net LED_BLUE: now also RN2.2 (R2.1), RN3.2 (R2.1)
- net LED_GREEN: now also RN2.1 (R1.1), RN3.1 (R1.1)
- net LED_RED: now also RN2.3 (R3.1), RN3.3 (R3.1)
- net P0.18/SWO: no longer J2.6 (Pin_6)
- net SWDCLK: now also U7.W31 (SWDCLK)
- net SWDIO: now also U7.AA31 (SWDIO)
- net VCC: now also C28.1, C29.1, C30.1, C31.1, C32.1, C33.1, C34.1, C35.1, C36.1, C37.1, C39.1, D2.1 (A), D4.1 (A), U7.A19 (VDD1), U7.AC1 (VDD), U7.AG1 (VDD), U7.AJ31 (VDD), U7.AL11 (VDD), U7.AL17 (VDD), U7.AL25 (VDD), U7.AL3 (VDD), U7.AL7 (VDD), U7.B28 (VDD), U7.B8 (VDD2), U7.C1 (VDD), U7.E31 (VDD), U7.N31 (VDD), U7.U1 (VDD)
- net at J1.1 (Pin_1): now also C46.1, L7.2
- net at C13.1, X2.1: now also U7.C31 (XC1)
- net at C10.1, X2.3: now also U7.B30 (XC2)
- net P0.00/XL1: no longer names the net of C11.2, X1.1
- net P0.00/XL1: now also U7.N1 (P0.00/XL1)
- net P0.01/XL2: no longer names the net of C12.2, X1.2
- net P0.01/XL2: now also U7.R1 (P0.01/XL2)
- net P0.11 renamed UART_TX
- net P0.12 renamed UART_RX
- net P0.25: no longer names the net of R13.1
- net P0.28 renamed PDM_CLK
- net P0.29 renamed PDM_DATA
- new net: L4.1, L6.2
- new net: L4.2, U7.B10 (DCCD)
- new net: D4.2 (BK), RN3.6 (R3.2)
- new net: D4.3 (GK), RN3.7 (R2.2)
- new net: D4.4 (RK), RN3.8 (R1.2)
- new net: C40.1, L6.1, U7.A15 (DECD)
- new net: D2.2 (BK), RN2.6 (R3.2)
- new net: D2.3 (GK), RN2.7 (R2.2)
- new net: D2.4 (RK), RN2.8 (R1.2)
- new net: C44.1, U7.A13 (DECA)
- new net: C38.1, C39(NP0)1.1, L5.1, U7.A27 (DECR), U7.G31 (DECRF)
- new net: C43.1, R20.2, U7.A5 (VBUS)
- new net: C41.2, U7.J1 (DCCH), U7.L1 (VDD3)
- new net: U7.A1 (NC), U7.A31 (NC), U7.AG31 (NC), U7.AL1 (NC), U7.AL31 (NC), U7.D2 (NC), U7.F2 (NC), U7.K2 (NC), U7.T2 (NC)
- new net: L3.1, L5.2
- new net: C42.1, U7.B6 (DECUSB)
- new net: L3.2, U7.A21 (DCC)
- new net: C45.1, U7.A23 (DECN)
- new net ANTENNA: C47.1, L7.1, U7.L31 (ANT)
- new net N_RESET: U7.AC31 (~{RESET})
- new net SWO: J2.6 (Pin_6)
- new net VBUS: R20.1
- no-connect marks 12 -> 9
Other:
- moved on the sheet: C15, C17, C18, C24, C25, D1, H1, H2, J2, MK1, R12, R13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

Commit message: saving the changes
Parts:
- MK1: value SPM1423HM4H -> CMM-4737DT
Changed lines of the file:
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@@
       (effects (font (size 1.27 1.27)) (justify right))
     )
-    (property "Value" "SPM1423HM4H" (at 29.1084 184.658 0)
+    (property "Value" "CMM-4737DT" (at 29.1084 184.658 0)
       (effects (font (size 1.27 1.27)) (justify right))
     )
@@
       (effects (font (size 1.27 1.27) italic) (justify left) hide)
     )
-    (property "Datasheet" "https://media.digikey.com/pdf/Data%20Sheets/Knowles%20Acoustics%20PDFs/SPM1423HM4H-B.pdf" (at 37.465 183.515 0)
+    (property "Datasheet" "https://www.digikey.com/en/products/detail/cui-devices/CMM-4737DT-26386-TR/9748843" (at 37.465 183.515 0)
       (effects (font (size 1.27 1.27)) hide)
     )
+    (property "Populate" "" (at 37.465 183.515 0)
+      (effects (font (size 1.27 1.27)) hide)
+    )

Commit message: saving changes: layout looks good, most DRC errors are fixed
Parts:
- removed D1, D2: ASMB-LTC2-0A335, nRF52832_qfaa:LED_Cree-PLCC4_2x2mm_CW, symbol LED:ASMB-MTB0-0A3A2
- removed J2: Conn_02x05_Odd_Even, Connector_PinHeader_1.27mm:PinHeader_2x05_P1.27mm_Vertical_SMD, symbol Connector_Generic:Conn_02x05_Odd_Even
- removed RN1, RN2: R_Pack04, Resistor_SMD:R_Array_Convex_4x0402, symbol Device:R_Pack04
- added C4: 100n, Capacitor_SMD:C_0201_0603Metric, symbol Device:C
- added D5: D_Schottky, Diode_SMD:D_SOD-123F, symbol Device:D_Schottky
- added J5: Conn_01x03_Socket, _other:JST_SM03B-SRSS-TB_LF__SN_, symbol Connector:Conn_01x03_Socket
- added R21: 1.6K, Resistor_SMD:R_0402_1005Metric, symbol Device:R
- added TP1, TP11, TP15, TP17, TP20, TP21, TP22, TP23, TP29, TP3, TP30, TP31: TestPoint, TestPoint:TestPoint_Pad_D1.0mm, symbol Connector:TestPoint
- R12: value 33 -> 330; LCSC C25105 -> C25104
- R13: value 330 -> 1K; LCSC C25104 -> C11702
Connections:
- net RTC_INT_N is gone; now on net WAKEUP_RTC: R12.1
- net UART_RX is gone; now on net DBG_RX: TP6.1
- net UART_TX is gone; now on net DBG_TX: TP7.1
- net GND: now also J3.5 (GND), J3.6 (Shield), C4.2, J5.1 (Pin_1), R21.2, TP23.1, TP29.1
- net I2C_SCL: now also U7.AE1 (P1.02/TWI)
- net I2C_SDA: now also U7.AF2 (P1.03/TWI)
- net LED_BLUE: now also U7.AK14 (P0.18/CSN)
- net LED_GREEN: now also U7.AL15 (P0.21)
- net LED_RED: now also U7.AL13 (P0.19)
- net MCU_POWER_LATCH: now also U7.R31 (P1.10)
- net MEM_CLK: now also U7.AL29 (P0.26/AIN5)
- net MEM_CS: now also U7.U31 (P0.29)
- net MEM_DI: now also U7.AK30 (P0.27/AIN6)
- net MEM_DO: now also U7.AE31 (P0.28/AIN7)
- net MEM_IO2: now also U7.AL23 (P1.08)
- net MEM_IO3: now also U7.AL27 (P0.24)
- net N_RESET: now also TP11.1, TP20.1
- net PDM_CLK: now also U7.AL9 (P0.16/IO[3])
- net PDM_DATA: now also U7.AL5 (P0.13/IO[0])
- net SWDCLK: now also TP17.1, TP3.1
- net SWDIO: now also TP1.1, TP15.1
- net VBAT_LEVEL: now also U7.V2 (P0.04/AIN0)
- net VBUS: now also J3.1 (VBUS)
- net VCC: now also TP21.1, TP22.1
- net DBG_TX: now reaches U7.B14 (P1.15)
- net DBG_TX: now also J5.2 (Pin_2), TP30.1
- net DBG_RX: now reaches U7.B18 (P1.12)
- net DBG_RX: now also J5.3 (Pin_3), TP31.1
- net BUTTON_INPUT_MCU: now reaches R13.1
- net BUTTON_INPUT_MCU: now also U7.B24 (P0.30), C4.1, R21.1
- net WAKEUP_RTC: now reaches U7.AB2 (P0.06/AIN2)
- net MAIN_BUTTON renamed BUTTON_INPUT
- net BUTTON_INPUT: now also D5.2 (A)
- new net VREG_EN: D5.1 (K)
- no-connect marks 9 -> 3
Other:
- moved on the sheet: TP6, TP7, TP8

Commit message: finalizing 1.4, going for the dry run
Parts:
- added C5, C7, C8: 100n, Capacitor_SMD:C_0201_0603Metric, symbol Device:C
- added C6: 1u, Capacitor_SMD:C_0402_1005Metric, symbol Device:C
- added D1: PRTR5V0U2X, Package_TO_SOT_SMD:SOT-143, symbol Power_Protection:PRTR5V0U2X
- added FB1, FB2, FB3: FerriteBead, Inductor_SMD:L_0402_1005Metric, symbol Device:FerriteBead
- added Q1: PMOS, Package_TO_SOT_SMD:SOT-23, symbol Simulation_SPICE:PMOS
- added R22: 4.7k, Resistor_SMD:R_0402_1005Metric, symbol Device:R
- added R23: 1M, Resistor_SMD:R_0402_1005Metric, symbol Device:R
- added R24: 100K, Resistor_SMD:R_0402_1005Metric, symbol Device:R
- added TP32: TestPoint, TestPoint:TestPoint_Pad_D1.0mm, symbol Connector:TestPoint
- U2: value W25Q32JVZP -> W25Q128JWPIQ
Connections:
- net GND: now also C5.2, C6.2, C7.2, C8.2, D1.1 (GND), FB2.1, FB3.1, Q1.1 (D), R22.2; no longer J3.5 (GND), J3.6 (Shield)
- net VBUS: now also C7.1, D1.4 (VCC), FB1.2; no longer J3.1 (VBUS)
- net VSS: now also R23.1, R24.1
- net WAKEUP_RTC: now also Q1.3 (S), R24.2; no longer R12.1, U7.AB2 (P0.06/AIN2)
- net USB_N: now reaches J3.2 (D-)
- net USB_N: now also U7.B4 (D-), D1.2 (I/O1)
- net USB_P: now reaches J3.3 (D+)
- net USB_P: now also U7.B2 (D+), D1.3 (I/O2)
- new net: C8.1, FB2.2, J3.6 (Shield), R22.1
- new net: FB3.2, J3.5 (GND)
- new net: C5.1, C6.1, FB1.1, J3.1 (VBUS)
- new net RTC_INT_N: Q1.2 (G), R12.1, R23.2, TP32.1, U7.AB2 (P0.06/AIN2)
Other:
- moved on the sheet: J3

Commit message: fixed couple issues with DF 1.4 (FF_CLK not propagated, RTC_INTR output inverted)
Parts:
- R23: LCSC C140195 -> C226699
Connections:
- net FF_CLK: now reaches U7.AL19 (P1.04)
