File: pcb/nRF52832_qfaa.kicad_pcb (KiCad board)
At the start: 4 copper layers, 41.5 x 13 mm, 77 parts, among them J1 Conn_01x01_Female, J2 Conn_02x05_Odd_Even, U1 NRF52832, U2 W25Q32JVZP, U3 TLV75533PDBVR, U4 BQ24078RGTR, X1 32.768kHz, X2 32MHz

Commit message: [pcb] version 1.3 (#75)
Changes:
    LDO voltage regulator replaced with DC-DC (expected increase in efficiency)
    added small-footprint RTC chip
    analog latch for regulator EN pin replaced with a digital flip-flop

Fixture:
    added Raspberry Pico to the PCB
    added current measurement setup
    planning to reduce hardware in use to a single PCB
Parts:
- removed D2: BAS40-05,215, Package_TO_SOT_SMD:SOT-23
- removed TP15, TP17, TP20, TP21, TP22, TP23: TestPoint, TestPoint:TestPoint_Pad_D1.0mm
- added C24: 1uF, Capacitor_SMD:C_0402_1005Metric, F.Cu at (53.8, 38.5)
- added C25: 100nF, Capacitor_SMD:C_0402_1005Metric, F.Cu at (55.5, 37.5)
- added C26: 1uF, Capacitor_SMD:C_0402_1005Metric, F.Cu at (54.6, 30.2)
- added C27: 100nF, Capacitor_SMD:C_0402_1005Metric, F.Cu at (59.7, 40.2)
- added L1: 0.47uH, Inductor_SMD:L_1008_2520Metric, F.Cu at (68.1, 38.0)
- added R12: 33, Resistor_SMD:R_0402_1005Metric, F.Cu at (55.6, 36.6)
- added R14: 100k, Resistor_SMD:R_0402_1005Metric, F.Cu at (62.3, 40.1)
- added R15: 511k, Resistor_SMD:R_0402_1005Metric, F.Cu at (63.3, 40.1)
- added R16: 91k, Resistor_SMD:R_0402_1005Metric, F.Cu at (62.9, 38.5)
- added R17: 1.6K, Resistor_SMD:R_0402_1005Metric, F.Cu at (54.4, 32.1)
- added R18: 100K, Resistor_SMD:R_0402_1005Metric, F.Cu at (60.7, 40.2)
- added R19: 100K, Resistor_SMD:R_0402_1005Metric, F.Cu at (48.2, 29.4)
- added R2: 4.7k, Resistor_SMD:R_0402_1005Metric, F.Cu at (58.1, 41.0)
- added R4: 4.7k, Resistor_SMD:R_0402_1005Metric, F.Cu at (53.7, 40.6)
- added TP5: TestPoint, TestPoint:TestPoint_Pad_D1.0mm, B.Cu at (49.9, 40.8)
- added U5: RV-4162-C7, _other:IC_RV-4162-C7, F.Cu at (55.5, 39.8)
- added U6: SN74LVC1G79DBVT, Package_TO_SOT_SMD:SOT-23-5, F.Cu at (51.8, 30.7)
- C1, C2: value 10uF -> 22uF; footprint Capacitor_SMD:C_0402_1005Metric -> Capacitor_SMD:C_0603_1608Metric
- C23: value 100pF -> 10uF
- TP24, TP25, TP26, TP27, TP28: moved to B.Cu
- U3: value TLV75533PDBVR -> TPS63802DLAR; footprint Package_TO_SOT_SMD:SOT-23-5 -> _other:VREG_TPS63802DLAR
- moved TP19 22.9 mm to (34.7, 30.2)
- moved TP13 20.2 mm to (40.0, 40.7)
- moved C2 19.8 mm to (65.3, 39.9), turned to 180 degrees
- moved TP27 16.5 mm to (66.7, 29.7), turned to 180 degrees
- moved TP25 12.0 mm to (67.5, 40.4), turned to 180 degrees
- moved TP18 9.83 mm to (55.9, 39.4)
- moved TP28 9.32 mm to (46.6, 40.8), turned to 180 degrees
- moved TP24 8.51 mm to (63.2, 40.1), turned to 180 degrees
- moved TP6 6.60 mm to (52.6, 31.0), turned to 180 degrees
- moved TP12 6.31 mm to (55.5, 29.9)
- moved C21 5.64 mm to (65.7, 34.4), turned to -90 degrees
- moved TP14 4.48 mm to (56.6, 33.3)
- moved C1 4.36 mm to (65.5, 36.0), turned to 180 degrees
- moved C23 3.25 mm to (65.4, 40.9), turned to 180 degrees
- moved TP26 2.50 mm to (67.0, 37.2), turned to 180 degrees
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Connections:
- C1 pad 1: VCC -> VSS
- C23 pad 1: /Power/LDO_EN -> VCC
- R5 pad 1: /Power/LDO_EN -> /Power/FF_D
- TP12 pad 1: /MEM_DI -> /Power/FF_D
- TP13 pad 1: /MEM_CS -> FF_CLK
- TP14 pad 1: /MEM_DO -> /Power/FF_Q
- TP16 pad 1: /Power/LDO_EN -> MAIN_BUTTON
- TP18 pad 1: VSS -> /I2C_SDA
- U1 pad 19: /P0.16 -> /I2C_SDA
- U1 pad 20: /P0.17 -> /I2C_SCL
- U1 pad 38: unconnected-(U1-Pad38) -> FF_CLK
- U1 pad 43: unconnected-(U1-Pad43) -> /RTC_INT_N
- U3 pad 1: VSS -> MAIN_BUTTON
- U3 pad 3: /Power/LDO_EN -> GND
- U3 pad 4: GND -> Net-(R15-Pad2)
- U3 pad 5: VCC -> Net-(R14-Pad2)
Routing:
- net FF_CLK: track 0.00 -> 34.4 mm, vias 0 -> 2
- net /Power/FF_D: track 0.00 -> 24.8 mm, vias 0 -> 2
- net +BATT: track 30.8 -> 8.34 mm
- net /I2C_SCL: track 0.00 -> 21.9 mm, vias 0 -> 2
- net /I2C_SDA: track 0.00 -> 21.8 mm, vias 0 -> 2
- net /Power/LDO_EN: track 13.5 -> 0.00 mm, vias 3 -> 0
- net VSS: track 39.9 -> 51.1 mm, vias 4 -> 8
- net GND: track 122.1 -> 132.7 mm, vias 35 -> 41
- net /RTC_INT_N: track 0.00 -> 10.6 mm, vias 0 -> 2
- net Net-(R12-Pad2): track 0.00 -> 10.1 mm, vias 0 -> 2
- net /Power/FF_Q: track 0.00 -> 6.10 mm, vias 0 -> 2
- net MAIN_BUTTON: track 27.1 -> 33.1 mm, vias 4 -> 5
- net /P0.12: track 2.32 -> 7.98 mm
- net /MEM_CS: track 19.9 -> 15.6 mm
- net Net-(R15-Pad2): track 0.00 -> 3.32 mm
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- added copper zone on F.Cu, net VCC
Other:
- board text added: "Dictofun 1.3"
- board text removed: "Dictofun 1.2"
- board text removed: "gnd"
- board text removed: "rx"
- board text removed: "tx"
