File: pcb/dictofun.kicad_sch (KiCad schematic)
At the start: 92 parts, among them J1 Conn_01x01_Female, J3 USB_B_Micro, J5 Conn_01x03_Socket, Q1 PMOS, U2 W25Q128JWPIQ, U5 RV-4162-C7, U7 NRF5340-QKAA-R7, X1 32.768kHz, X2 32MHz

Commit message: Design Freeze DF 1.4
Parts:
- S1: footprint SW_KMR221GLFS -> df_components:SW_KMR221GLFS
Connections:
- net RTC_CLKOUT: no longer names the net of U5.2 (CLKOUT)
- no-connect marks 3 -> 34

Commit message: fixed error: RTC PFET could shorten battery to the ground
Parts:
- added R25: 330, Resistor_SMD:R_0402_1005Metric, symbol Device:R
Connections:
- net WAKEUP_RTC: now also R25.1; no longer Q1.3 (S), R24.2
- new net: Q1.3 (S), R24.2, R25.2
Changed lines of the file:
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@@
     (stroke (width 0) (type default))
   )
+  (wire (pts (xy 386.715 33.655) (xy 390.525 33.655))
+    (stroke (width 0) (type default))
+  )
   (wire (pts (xy 25.4 133.985) (xy 36.83 133.985))
     (stroke (width 0) (type default))
@@
     )
   )
-  (global_label "WAKEUP_RTC" (shape input) (at 379.095 33.655 0) (fields_autoplaced)
+  (global_label "WAKEUP_RTC" (shape input) (at 390.525 33.655 0) (fields_autoplaced)
     (effects (font (size 1.27 1.27)) (justify left))
-    (property "Intersheetrefs" "${INTERSHEET_REFS}" (at 393.4607 33.655 0)
+    (property "Intersheetrefs" "${INTERSHEET_REFS}" (at 404.8907 33.655 0)
       (effects (font (size 1.27 1.27)) (justify left) hide)
     )
@@
         )
       )
+    )
+  )
+  (symbol (lib_id "Device:R") (at 382.905 33.655 270) (unit 1)
+    (in_bom yes) (on_board yes) (dnp no)
+    (property "Reference" "R25" (at 382.27 31.75 90)
+      (effects (font (size 1.27 1.27)))
+    )
+    (property "Value" "330" (at 383.54 36.195 90)
+      (effects (font (size 1.27 1.27)))
+    )
+    (property "Footprint" "Resistor_SMD:R_0402_1005Metric" (at 382.905 31.877 90)
+      (effects (font (size 1.27 1.27)) hide)
+    )
+    (property "Datasheet" "~" (at 382.905 33.655 0)
+      (effects (font (size 1.27 1.27)) hide)
+    )
+    (property "LCSC" "C25104" (at 382.905 33.655 0)
+      (effects (font (size 1.27 1.27)) hide)
+    )
+    (property "Populate" "" (at 382.905 33.655 0)
+      (effects (font (size 1.27 1.27)) hide)
+    )
+    (pin "1")
+    (pin "2")
+    (instances
+      (project "dictofun"
+        (path "/109caac1-5036-4f23-9a66-f569d871501b"
+          (reference "R25") (unit 1)
+        )
+      )

Commit message: prepared the df1.4 fabrication outputs
Parts:
- C11: LCSC (none) -> C161369
- C47: LCSC (none) -> C384700
- L7: LCSC (none) -> C1329438
- U7: LCSC (none) -> C3015611
Changed lines of the file:
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@@
       (effects (font (size 1.27 1.27)) hide)
     )
-    (property "LCSC" "" (at 132.08 106.045 0)
+    (property "LCSC" "C161369" (at 132.08 106.045 0)
       (effects (font (size 1.27 1.27)) hide)
     )
@@
       (effects (font (size 1.27 1.27)) hide)
     )
+    (property "LCSC" "C3015611" (at 213.995 171.45 0)
+      (effects (font (size 1.27 1.27)) hide)
+    )
     (pin "B20")
     (pin "AL15")
@@
       (effects (font (size 1.27 1.27)) hide)
     )
-    (property "LCSC" "" (at 273.05 69.85 0)
+    (property "LCSC" "C384700" (at 273.05 69.85 0)
       (effects (font (size 1.27 1.27)) hide)
     )
@@
       (effects (font (size 1.27 1.27)) hide)
     )
+    (property "LCSC" "C3015611" (at 213.36 72.39 0)
+      (effects (font (size 1.27 1.27)) hide)
+    )
     (pin "B20")
     (pin "AL15")
@@
       (effects (font (size 1.27 1.27)) hide)
     )
+    (property "LCSC" "C3015611" (at 165.1 46.355 0)
+      (effects (font (size 1.27 1.27)) hide)
+    )
     (pin "B20")
     (pin "AL15")
@@
       (effects (font (size 1.27 1.27)) hide)
     )
+    (property "LCSC" "C3015611" (at 187.325 150.495 0)
+      (effects (font (size 1.27 1.27)) hide)
+    )
     (pin "B20")
     (pin "AL15")
@@
       (effects (font (size 1.27 1.27)) hide)
     )
-    (property "LCSC" "" (at 281.94 66.04 90)
+    (property "LCSC" "C1329438" (at 281.94 66.04 90)
       (effects (font (size 1.27 1.27)) hide)
     )

Commit message: fixed another issue (added current limiting resistor, added testpoint for button control)
Parts:
- added TP33: TestPoint, TestPoint:TestPoint_Pad_D1.0mm, symbol Connector:TestPoint
Connections:
- net BUTTON_INPUT: now also TP33.1
Changed lines of the file:
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@@
     (stroke (width 0) (type default))
   )
+  (wire (pts (xy 38.735 45.72) (xy 38.735 44.45))
+    (stroke (width 0) (type default))
+  )
   (wire (pts (xy 283.21 36.195) (xy 299.72 36.195))
     (stroke (width 0) (type default))
@@
     (stroke (width 0) (type default))
   )
-  (wire (pts (xy 43.18 45.72) (xy 60.96 45.72))
+  (wire (pts (xy 38.735 45.72) (xy 60.96 45.72))
     (stroke (width 0) (type default))
   )
@@
         )
       )
+    )
+  )
+  (symbol (lib_id "Connector:TestPoint") (at 38.735 44.45 0) (unit 1)
+    (in_bom yes) (on_board yes) (dnp no)
+    (property "Reference" "TP33" (at 40.2082 42.6212 0)
+      (effects (font (size 1.27 1.27)) (justify left))
+    )
+    (property "Value" "TestPoint" (at 40.2082 43.7642 0)
+      (effects (font (size 1.27 1.27)) (justify left) hide)
+    )
+    (property "Footprint" "TestPoint:TestPoint_Pad_D1.0mm" (at 43.815 44.45 0)
+      (effects (font (size 1.27 1.27)) hide)
+    )
+    (property "Datasheet" "~" (at 43.815 44.45 0)
+      (effects (font (size 1.27 1.27)) hide)
+    )
+    (pin "1")
+    (instances
+      (project "dictofun"
+        (path "/109caac1-5036-4f23-9a66-f569d871501b"
+          (reference "TP33") (unit 1)
+        )
+      )

Commit message: df 1.4.52840 ready for production
Parts:
- removed C13: 10pF, Capacitor_SMD:C_0402_1005Metric, symbol nRF52832_qfaa-eagle-import:CAPACITOR_0402_N
- removed C30, C31, C32, C33, C34, C35, C45: 100n, Capacitor_SMD:C_0201_0603Metric, symbol Device:C
- removed C36: N.C, Capacitor_SMD:C_0201_0603Metric, symbol Device:C
- removed C37, C38, C39, C40, C44: 1u, Capacitor_SMD:C_0402_1005Metric, symbol Device:C
- removed C39(NP0)1: 100pF, Capacitor_SMD:C_0201_0603Metric, symbol Device:C
- removed C41: 2.2u, Capacitor_SMD:C_0603_1608Metric, symbol Device:C
- removed C42, C43: 4.7u, Capacitor_SMD:C_0603_1608Metric, symbol Device:C
- removed L4: 10uH, Inductor_SMD:L_0603_1608Metric, symbol Device:L
- removed L5, L6: 15nH, Inductor_SMD:L_0201_0603Metric, symbol Device:L
- removed R20: 4.7, Resistor_SMD:R_0201_0603Metric, symbol Device:R
- removed TP11, TP20, TP30, TP31: TestPoint, TestPoint:TestPoint_Pad_D1.0mm, symbol Connector:TestPoint
- removed U7: NRF5340-QKAA-R7, _other:XCVR_NRF5340-QKAA-R7, symbol NRF5340:NRF5340-QKAA-R7
- added C13, C22, C53, C54: 100nF, Capacitor_SMD:C_0402_1005Metric, symbol Device:C
- added C14, C55: 1uF, Capacitor_SMD:C_0402_1005Metric, symbol Device:C
- added C16, C48: N.C, Capacitor_SMD:C_0402_1005Metric, symbol Device:C
- added C49: 820pF, Capacitor_SMD:C_0402_1005Metric, symbol Device:C
- added C50, C51, C52: 4.7uF, Capacitor_SMD:C_0603_1608Metric, symbol Device:C
- added C9: 10pF, Capacitor_SMD:C_0402_1005Metric, symbol nRF52832_qfaa-eagle-import:CAPACITOR_0402_N
- added L2: 10uH, Inductor_SMD:L_0402_1005Metric, symbol Device:L
- added U1: nRF52840, Package_DFN_QFN:Nordic_AQFN-73-1EP_7x7mm_P0.5mm, symbol MCU_Nordic:nRF52840
- C11: footprint Capacitor_SMD:C_0201_0603Metric -> Capacitor_SMD:C_0402_1005Metric; LCSC C161369 -> C32949
- C12: footprint Capacitor_SMD:C_0201_0603Metric -> Capacitor_SMD:C_0402_1005Metric; LCSC (none) -> C32949
- C17, C24: LCSC C52923 -> C77007
- C28: value 100n -> 100p; footprint Capacitor_SMD:C_0201_0603Metric -> Capacitor_SMD:C_0402_1005Metric; LCSC C5142565 -> C445763
- C29: value 100n -> 47nF; footprint Capacitor_SMD:C_0201_0603Metric -> Capacitor_SMD:C_0402_1005Metric; LCSC C5142565 -> C338148
- C4, C5, C7, C8: value 100n -> 100nF; footprint Capacitor_SMD:C_0201_0603Metric -> Capacitor_SMD:C_0402_1005Metric; LCSC C5142565 -> C1525
- C46: footprint Capacitor_SMD:C_0201_0603Metric -> Capacitor_SMD:C_0402_1005Metric
- C47: footprint Capacitor_SMD:C_0201_0603Metric -> Capacitor_SMD:C_0402_1005Metric; LCSC C384700 -> C2194394
- C6: value 1u -> 1uF
- L3: value 10uH -> 15nH; footprint Inductor_SMD:L_0603_1608Metric -> Inductor_SMD:L_0402_1005Metric; LCSC C5339208 -> (none)
- L7: footprint Inductor_SMD:L_0201_0603Metric -> Inductor_SMD:L_0402_1005Metric; LCSC C1329438 -> (none)
- X2: footprint nRF52832_qfaa:BT-XTAL_2016_N -> df_components:BT-XTAL_2016_N
Connections:
- net ANTENNA: now also U1.H23 (ANT)
- net BUTTON_INPUT_MCU: now also U1.A16 (P1.13)
- net DBG_RX: now also U1.L1 (P0.06)
- net DBG_TX: now also U1.J1 (AIN2/P0.04)
- net FF_CLK: now also U1.A14 (P1.15)
- net GND: now also C13.2, C14.2, C16.2, C22.2, C48.2, C49.2, C50.2, C51.2, C52.2, C53.2, C54.2, C55.2, C9.2, U1.B7 (VSS), U1.EP (VSS), U1.F23 (VSS_PA)
- net I2C_SCL: now also U1.R1 (TRACEDATA3/P1.09)
- net I2C_SDA: now also U1.U1 (TRACEDATA1/P0.12)
- net LED_BLUE: now also U1.AD20 (P0.24)
- net LED_GREEN: now also U1.AD22 (TRACEDATA0/P1.00)
- net LED_RED: now also U1.AD18 (P0.22)
- net MCU_POWER_LATCH: now also U1.A12 (AIN0/P0.02)
- net MEM_CLK: now also U1.P23 (P1.07)
- net MEM_CS: now also U1.R24 (P1.06)
- net MEM_DI: now also U1.W24 (P1.02)
- net MEM_DO: now also U1.U24 (P1.04)
- net MEM_IO2: now also U1.L24 (NFC1/P0.09)
- net MEM_IO3: now also U1.AC21 (P0.25)
- net N_RESET: now also U1.AC13 (P0.18/~{RESET})
- net PDM_CLK: now also U1.AD10 (P0.15)
- net PDM_DATA: now also U1.AD12 (P0.17)
- net RTC_INT_N: now also U1.N1 (P0.08)
- net SWDCLK: now also U1.AA24 (SWDCLK)
- net SWDIO: now also U1.AC24 (SWDIO)
- net USB_N: now also U1.AD4 (D-)
- net USB_P: now also U1.AD6 (D+)
- net VBAT_LEVEL: now also U1.A10 (AIN5/P0.29)
- net VBUS: now also C51.1, U1.AD2 (VBUS)
- net VCC: now also C22.1, C52.1, C53.1, C54.1, C55.1, U1.A22 (VDD), U1.AD14 (VDD), U1.AD23 (VDD), U1.B1 (VDD), U1.W1 (VDD), U1.Y2 (VDDH); no longer C28.1, C29.1
- net at C11.2, X1.1: now also U1.F2 (XL2/P0.01)
- net at C12.2, X1.2: now also U1.D2 (XL1/P0.00)
- net at X2.1: now also C10.1, U1.B24 (XC1)
- net at X2.3: now also C9.1, U1.A23 (XC2); no longer C10.1
- net DEC4: now reaches L3.1
- net DEC4: now also C29.1, L3.2, C14.1, C48.1, L2.2, U1.B5 (DEC4), U1.E24 (DEC6)
- new net DCC: L2.1, U1.B3 (DCC)
- new net DCCH: U1.AB2 (DCCH)
- new net DEC1: C13.1, U1.C1 (DEC1)
- new net DEC2: C16.1, U1.A18 (DEC2)
- new net DEC3: C28.1, U1.D23 (DEC3)
- new net DEC5: C49.1, U1.N24 (DEC5)
- new net DECUSB: C50.1, U1.AC5 (DECUSB)
- no-connect marks 34 -> 6
Other:
- note added: "Using reference circuit #5 from the reference manual"
- moved on the sheet: D4, H1, H2, J5, RN3, TP1, TP15, TP17, TP21, TP22, TP23, TP29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

Commit message: fixing the state of harness for 1.4.52840
Parts:
- L7: LCSC (none) -> C97985
- U1: LCSC (none) -> C190794
Changed lines of the file:
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@@
+      (effects (font (size 1.27 1.27)) hide)
+    )
+    (property "LCSC" "C190794" (at 173.99 113.03 0)
       (effects (font (size 1.27 1.27)) hide)
     )
@@
       (effects (font (size 1.27 1.27)) hide)
     )
-    (property "LCSC" "" (at 281.94 66.04 90)
+    (property "LCSC" "C97985" (at 281.94 66.04 90)
       (effects (font (size 1.27 1.27)) hide)
     )
