File: pcb/test_fixture/v1.4/rp2040_and_shifters.kicad_sch (KiCad schematic)
At the start: 16 parts, among them U1 SC0915, U4 SN74AVC4T774RSVR, U5 TXB0104RGY, U6 SN74AVC4T774RSVR, U7 SN74AVC4T774RSVR

Commit message: v1.4.52840 harness done
Parts:
- removed R9: 1K, Resistor_SMD:R_0603_1608Metric, symbol Device:R
- added J1: SM03B-SRSS-TB_LF__SN_, df_footprints:JST_SM03B-SRSS-TB_LF__SN_, symbol SM03B-SRSS-TB_LF__SN_:SM03B-SRSS-TB_LF__SN_
- added OE_CTRL_TP1: (no value), TestPoint:TestPoint_Pad_D1.5mm, symbol Connector:TestPoint
Connections:
- net BUTTON_CTRL: now also U1.9 (GP6); no longer U6.11 (B2), U6.2 (A2)
- net GND: now also J1.1, J1.S1 (SHIELD), J1.S2 (SHIELD)
- net OE_CTRL: now also OE_CTRL_TP1.1
- net SWDIO: no longer U5.13 (B1)
- net UART_RX: now also J1.3
- net UART_TX: now also J1.2
- new net SWDIO_1.8: U5.13 (B1)
