File: pcb/test_fixture/v1.4/test_fixture.kicad_pcb (KiCad board)
At the start: 2 copper layers, 71.5 x 74.9 mm, 71 parts, among them J2 SM03B-SRSS-TB_LF__SN_, J3 Conn_ARM_JTAG_SWD_10, Q1 NMOS, SW1 SW_SPDT, U1 SC0915, U2 MIC29302WU, U3 INA186A5IDCKR, U4 SN74AVC4T774RSVR, U5 TXB0104RGY, U6 SN74AVC4T774RSVR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

Commit message: v1.4.52840 harness done
Parts:
- removed C1, C4: 1u, Resistor_SMD:R_1206_3216Metric
- removed C5, C8: 100n, Resistor_SMD:R_1206_3216Metric
- removed J2: SM03B-SRSS-TB_LF__SN_, df_footprints:JST_SM03B-SRSS-TB_LF__SN_
- removed JP5: Jumper_2_Bridged, Jumper:SolderJumper-2_P1.3mm_Bridged2Bar_Pad1.0x1.5mm
- removed POGO13: pogo, fixture:POGO
- removed R3: 0.04, Resistor_SMD:R_Shunt_Vishay_WSR2_WSR3_KelvinConnection
- removed R9: 1K, Resistor_SMD:R_0603_1608Metric
- removed U3: INA186A5IDCKR, df_footprints:SOT65P210X110-6N
- added GND1: , TestPoint:TestPoint_Pad_D1.5mm, F.Cu at (101.8, 94.5)
- added GND2: , TestPoint:TestPoint_Pad_D1.5mm, F.Cu at (149.6, 113.2)
- added GND3: , TestPoint:TestPoint_Pad_D1.5mm, F.Cu at (89.0, 98.2)
- added J1: SM03B-SRSS-TB_LF__SN_, df_footprints:JST_SM03B-SRSS-TB_LF__SN_, F.Cu at (88.2, 82.7)
- added OE_CTRL_TP1: , TestPoint:TestPoint_Pad_D1.5mm, F.Cu at (148.0, 109.9)
- moved SW1 21.3 mm to (109.2, 113.8)
- moved C9 21.3 mm to (101.7, 116.3)
- moved FF_Q1 16.9 mm to (143.4, 99.4)
- moved C10 11.5 mm to (103.5, 103.0), turned to 180 degrees
- moved R6 10.1 mm to (132.3, 99.5)
- moved R5 7.39 mm to (130.7, 99.5), turned to 90 degrees
- moved BUTTON1 5.70 mm to (147.1, 115.9)
- moved Q1 2.36 mm to (122.8, 108.9)
- moved R10 2.36 mm to (122.7, 112.4)
- moved R4 2.36 mm to (122.7, 114.7)
- moved R1 1.33 mm to (96.3, 100.5), turned to -90 degrees
- moved R2 1.33 mm to (98.9, 100.5)
- moved POGO7 0.13 mm to (133.1, 88.1)
Connections:
- BATT+1 pad 1: /BATT+ -> VDD
- FF_Q1 pad 1: /FF_Q -> FF_Q_1.8
- J3 pad 1: VREF_IN -> VREF_IN_1.8
- POGO15 pad 1: /FF_Q -> FF_Q_1.8
- POGO19 pad 1: /BATT+ -> VDD
- POGO2 pad 1: VREF_IN -> VREF_IN_1.8
- U1 pad 6: SWDIO -> /RP2040 and Shifters/SWDIO
- U1 pad 9: Net-(U1-GP6) -> BUTTON_CTRL
- U5 pad 13: SWDIO -> SWDIO_1.8
- U5 pad 2: SWDIO -> /RP2040 and Shifters/SWDIO
- U6 pad 11: BUTTON_CTRL -> unconnected-(U6-B2-Pad11)
- U6 pad 2: BUTTON_CTRL -> unconnected-(U6-A2-Pad2)
Routing:
- net GND: track 0.00 -> 189.5 mm, vias 0 -> 49
- net /RP2040 and Shifters/UART_TX: track 0.00 -> 119.8 mm, vias 0 -> 4
- net /RP2040 and Shifters/UART_RX: track 0.00 -> 111.7 mm, vias 0 -> 4
- net VDD: track 0.00 -> 104.0 mm, vias 0 -> 7
- net +3.3V: track 0.00 -> 94.6 mm, vias 0 -> 7
- net +1.8V: track 0.00 -> 78.6 mm, vias 0 -> 4
- net VREF_IN_1.8: track 0.00 -> 77.0 mm, vias 0 -> 5
- net /UART_TX_TO_MCU_1.8: track 0.00 -> 64.7 mm, vias 0 -> 3
- net I2C_CLK_1.8: track 0.00 -> 62.3 mm, vias 0 -> 3
- net /I2C_DATA_1.8: track 0.56 -> 61.2 mm
- net /BUTTON: track 0.00 -> 53.8 mm
- net SWDCLK_1.8: track 0.00 -> 52.6 mm, vias 0 -> 1
- net /RP2040 and Shifters/SWDIO: track 0.00 -> 49.2 mm, vias 0 -> 3
- net /RP2040 and Shifters/SWDCLK: track 0.00 -> 49.0 mm, vias 0 -> 2
- net /RP2040 and Shifters/RESET: track 0.00 -> 47.9 mm, vias 0 -> 2
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- added copper zone on In1.Cu, net +1.8V
- added copper zone on In2.Cu, net GND
Other:
- copper layers 2 -> 4
- board text added: "1.8"
- board text added: "BTN"
- board text added: "FF_CK"
- board text added: "FF_D"
- board text added: "FF_Q"
- board text added: "GND"
- board text added: "I2CC"
- board text added: "I2CD"
- board text added: "OE"
- board text added: "VBAT"
- board text added: "v1.4.52840"

Commit message: Saving the first iteration of harness outputs
Changed lines of the file:
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@@
       (drillshape 0)
       (scaleselection 1)
-      (outputdirectory "../out/v1.3_fixture/gerber")
+      (outputdirectory "../../out/v1.4_fixture/gerbers/")
     )
   )
@@
     (fp_circle (center 0 0) (end 2.35 0)
       (stroke (width 0.05) (type solid)) (fill none) (layer "F.CrtYd"))
-    (pad "" np_thru_hole circle locked (at 0 0) (size 2.1 2.1) (drill 2.1) (layers "*.Cu" "*.Mask"))
+    (pad "" np_thru_hole circle (at 0 0) (size 2.1 2.1) (drill 2.1) (layers "*.Cu" "*.Mask"))
   )
   (footprint "fixture:POGO" locked (layer "F.Cu")
@@
     (fp_circle (center 0 0) (end 2.35 0)
       (stroke (width 0.05) (type solid)) (fill none) (layer "F.CrtYd"))
-    (pad "" np_thru_hole circle locked (at 0 0) (size 2.1 2.1) (drill 2.1) (layers "*.Cu" "*.Mask"))
+    (pad "" np_thru_hole circle (at 0 0) (size 2.1 2.1) (drill 2.1) (layers "*.Cu" "*.Mask"))
   )
   (footprint "Package_DFN_QFN:Texas_S-PVQFN-N14" (layer "F.Cu")
@@
     (fp_line (start 5.625 5) (end 4.625 5)
       (stroke (width 0.1) (type solid)) (layer "F.Fab"))
-    (pad "1" smd roundrect (at -7.65 -3.4 180) (size 4.6 1.1) (layers "F.Cu" "F.Paste" "F.Mask") (roundrect_rratio 0.227273)
+    (pad "1" smd roundrect (at -7.65 -3.4 180) (size 4.6 1.1) (layers "F.Cu" "F.Paste" "F.Mask") (roundrect_rratio 0.2272727273)
       (net 8 "+5V") (pinfunction "EN") (pintype "input"))
-    (pad "2" smd roundrect (at -7.65 -1.7 180) (size 4.6 1.1) (layers "F.Cu" "F.Paste" "F.Mask") (roundrect_rratio 0.227273)
+    (pad "2" smd roundrect (at -7.65 -1.7 180) (size 4.6 1.1) (layers "F.Cu" "F.Paste" "F.Mask") (roundrect_rratio 0.2272727273)
       (net 8 "+5V") (pinfunction "VIN") (pintype "power_in"))
-    (pad "3" smd roundrect (at -7.65 0 180) (size 4.6 1.1) (layers "F.Cu" "F.Paste" "F.Mask") (roundrect_rratio 0.227273)
+    (pad "3" smd roundrect (at -7.65 0 180) (size 4.6 1.1) (layers "F.Cu" "F.Paste" "F.Mask") (roundrect_rratio 0.2272727273)
       (net 4 "GND") (pinfunction "GND") (pintype "power_in"))
-    (pad "3" smd roundrect (at -0.925 -2.775 180) (size 4.55 5.25) (layers "F.Cu" "F.Paste") (roundrect_rratio 0.054945)
+    (pad "3" smd roundrect (at -0.925 -2.775 180) (size 4.55 5.25) (layers "F.Cu" "F.Paste") (roundrect_rratio 0.05494505495)
       (net 4 "GND") (pinfunction "GND") (pintype "power_in"))
-    (pad "3" smd roundrect (at -0.925 2.775 180) (size 4.55 5.25) (layers "F.Cu" "F.Paste") (roundrect_rratio 0.054945)
+    (pad "3" smd roundrect (at -0.925 2.775 180) (size 4.55 5.25) (layers "F.Cu" "F.Paste") (roundrect_rratio 0.05494505495)
       (net 4 "GND") (pinfunction "GND") (pintype "power_in"))
-    (pad "3" smd roundrect (at 1.5 0 180) (size 9.4 10.8) (layers "F.Cu" "F.Mask") (roundrect_rratio 0.026596)
+    (pad "3" smd roundrect (at 1.5 0 180) (size 9.4 10.8) (layers "F.Cu" "F.Mask") (roundrect_rratio 0.02659595745)
       (net 4 "GND") (pinfunction "GND") (pintype "power_in"))
-    (pad "3" smd roundrect (at 3.925 -2.775 180) (size 4.55 5.25) (layers "F.Cu" "F.Paste") (roundrect_rratio 0.054945)
+    (pad "3" smd roundrect (at 3.925 -2.775 180) (size 4.55 5.25) (layers "F.Cu" "F.Paste") (roundrect_rratio 0.05494505495)
       (net 4 "GND") (pinfunction "GND") (pintype "power_in"))
-    (pad "3" smd roundrect (at 3.925 2.775 180) (size 4.55 5.25) (layers "F.Cu" "F.Paste") (roundrect_rratio 0.054945)
+    (pad "3" smd roundrect (at 3.925 2.775 180) (size 4.55 5.25) (layers "F.Cu" "F.Paste") (roundrect_rratio 0.05494505495)
       (net 4 "GND") (pinfunction "GND") (pintype "power_in"))
-    (pad "4" smd roundrect (at -7.65 1.7 180) (size 4.6 1.1) (layers "F.Cu" "F.Paste" "F.Mask") (roundrect_rratio 0.227273)
+    (pad "4" smd roundrect (at -7.65 1.7 180) (size 4.6 1.1) (layers "F.Cu" "F.Paste" "F.Mask") (roundrect_rratio 0.2272727273)
       (net 9 "VDD") (pinfunction "VOUT") (pintype "power_out"))
-    (pad "5" smd roundrect (at -7.65 3.4 180) (size 4.6 1.1) (layers "F.Cu" "F.Paste" "F.Mask") (roundrect_rratio 0.227273)
+    (pad "5" smd roundrect (at -7.65 3.4 180) (size 4.6 1.1) (layers "F.Cu" "F.Paste" "F.Mask") (roundrect_rratio 0.2272727273)
       (net 12 "Net-(U2-ADJ)") (pinfunction "ADJ") (pintype "input"))
     (model "${KICAD6_3DMODEL_DIR}/Package_TO_SOT_SMD.3dshapes/TO-263-5_TabPin3.wrl"
@@
     (fp_circle (center 0 0) (end 2.35 0)
       (stroke (width 0.05) (type solid)) (fill none) (layer "F.CrtYd"))
-    (pad "" np_thru_hole circle locked (at 0 0) (size 2.1 2.1) (drill 2.1) (layers "*.Cu" "*.Mask"))
+    (pad "" np_thru_hole circle (at 0 0) (size 2.1 2.1) (drill 2.1) (layers "*.Cu" "*.Mask"))
   )
   (footprint "Capacitor_SMD:C_0402_1005Metric" (layer "F.Cu")
@@
     (fp_circle (center 0 0) (end 2.35 0)
       (stroke (width 0.05) (type solid)) (fill none) (layer "F.CrtYd"))
-    (pad "" np_thru_hole circle locked (at 0 0) (size 2.1 2.1) (drill 2.1) (layers "*.Cu" "*.Mask"))
+    (pad "" np_thru_hole circle (at 0 0) (size 2.1 2.1) (drill 2.1) (layers "*.Cu" "*.Mask"))
   )
   (footprint "fixture:POGO" locked (layer "F.Cu")
@@
     (fp_line (start 1.6 0.8) (end -1.6 0.8)
       (stroke (width 0.1) (type solid)) (layer "F.Fab"))
-    (pad "1" smd roundrect (at -1.475 0 180) (size 1.15 1.8) (layers "F.Cu" "F.Paste" "F.Mask") (roundrect_rratio 0.217391)
+    (pad "1" smd roundrect (at -1.475 0 180) (size 1.15 1.8) (layers "F.Cu" "F.Paste" "F.Mask") (roundrect_rratio 0.2173913043)
       (net 9 "VDD") (pintype "passive"))
-    (pad "2" smd roundrect (at 1.475 0 180) (size 1.15 1.8) (layers "F.Cu" "F.Paste" "F.Mask") (roundrect_rratio 0.217391)
+    (pad "2" smd roundrect (at 1.475 0 180) (size 1.15 1.8) (layers "F.Cu" "F.Paste" "F.Mask") (roundrect_rratio 0.2173913043)
       (net 4 "GND") (pintype "passive"))
     (model "${KICAD6_3DMODEL_DIR}/Capacitor_SMD.3dshapes/C_1206_3216Metric.wrl"
@@
     (fp_line (start 1.6 0.8) (end -1.6 0.8)
       (stroke (width 0.1) (type solid)) (layer "F.Fab"))
-    (pad "1" smd roundrect (at -1.4625 0) (size 1.125 1.75) (layers "F.Cu" "F.Paste" "F.Mask") (roundrect_rratio 0.222222)
+    (pad "1" smd roundrect (at -1.4625 0) (size 1.125 1.75) (layers "F.Cu" "F.Paste" "F.Mask") (roundrect_rratio 0.2222222222)
       (net 8 "+5V") (pintype "passive"))
-    (pad "2" smd roundrect (at 1.4625 0) (size 1.125 1.75) (layers "F.Cu" "F.Paste" "F.Mask") (roundrect_rratio 0.222222)
+    (pad "2" smd roundrect (at 1.4625 0) (size 1.125 1.75) (layers "F.Cu" "F.Paste" "F.Mask") (roundrect_rratio 0.2222222222)
       (net 4 "GND") (pintype "passive"))
     (model "${KICAD6_3DMODEL_DIR}/Resistor_SMD.3dshapes/R_1206_3216Metric.wrl"
