File: pcb/test_fixture/test_fixture.kicad_pcb (KiCad board)
At the start: 2 copper layers, 71.5 x 74.9 mm, 80 parts, among them J1 UART, J3 Conn_ARM_JTAG_SWD_10, J5 GND, J6 GND, P3.3V1 , U1 SC0915, U2 MIC29302WU, U3 INA186A5IDCKR, U4 INA186A5IDCKR

Commit message: PCB v1.4 (#175)
Parts:
- removed C2, C3: 1u, Resistor_SMD:R_1206_3216Metric
- removed C6, C7: 100n, Resistor_SMD:R_1206_3216Metric
- removed DEC_CAP1, GND1, GND2, PDM_CLK1, PDM_DATA1: , TestPoint:TestPoint_Pad_D1.5mm
- removed J5, J6: GND, fixture:POGO
- removed JP2, JP4, JP7, JP8: Jumper_2_Open, Jumper:SolderJumper-2_P1.3mm_Open_RoundedPad1.0x1.5mm
- removed POGO17, POGO18, POGO20, POGO23, POGO24, POGO25, POGO4: pogo, fixture:POGO
- removed U4: INA186A5IDCKR, fixture:SOT65P210X110-6N
- added Q1: NMOS, Package_TO_SOT_SMD:SOT-23, F.Cu at (163.3, 110.3)
- added R10: 1K, Resistor_SMD:R_0603_1608Metric, F.Cu at (162.9, 116.3)
- R4: value 0.01 -> 100K; footprint Resistor_SMD:R_Shunt_Vishay_WSR2_WSR3_KelvinConnection -> Resistor_SMD:R_0603_1608Metric
- moved H8 58.0 mm to (161.1, 85.5)
- moved H7 57.6 mm to (161.1, 79.8)
- moved R9 43.3 mm to (171.6, 111.0), turned to 0 degrees
- moved R7 38.3 mm to (171.6, 105.9)
- moved R8 35.7 mm to (171.6, 108.5)
- moved R5 27.9 mm to (171.6, 100.9)
- moved R4 27.3 mm to (162.9, 113.7)
- moved R6 25.3 mm to (171.6, 103.4)
- moved POGO3 24.5 mm to (131.4, 82.3)
- moved POGO16 20.8 mm to (126.1, 78.4)
- moved POGO12 20.3 mm to (112.9, 80.2)
- moved H9 18.3 mm to (161.1, 91.2)
- moved POGO6 18.0 mm to (139.2, 92.3)
- moved FF_CLK1 17.6 mm to (130.8, 100.9)
- moved POGO14 16.9 mm to (119.5, 95.2)
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- renumbered P3.3V1 to VCC_SENSE1
Connections:
- J3 pad 10: /RESET -> unconnected-(J3-~{RESET}-Pad10)
- J3 pad 6: /SWO -> unconnected-(J3-SWO/TDO-Pad6)
- J3 pad 8: Net-(J3-Pad8) -> unconnected-(J3-NC/TDI-Pad8)
- J3 pad 9: GND -> unconnected-(J3-GNDDetect-Pad9)
- POGO16 pad 1: /P3.3V -> /P1.9V
- R4 pad 1: Net-(JP7-Pad2) -> /BUTTON_CTRL
- R4 pad 2: /BATT+ -> GND
- R5 pad 1: /P3.3V -> /VCC_SENSE
- R5 pad 2: /SENSE_3_3V -> /SENSE_VCC
- R6 pad 1: /SENSE_3_3V -> /SENSE_VCC
- R9 pad 1: /BUTTON -> /BUTTON_CTRL
- U1 pad 32: /DEC_CAP -> unconnected-(U1-GP27-Pad32)
- VCC_SENSE1 pad 1: /P3.3V -> /P1.9V
Routing:
- net /PDM_DATA: track 114.3 -> 44.7 mm, vias 1 -> 0
- net /BATT+: track 72.9 -> 8.07 mm
- net /I2C_CLK: track 92.3 -> 32.1 mm, vias 2 -> 1
- net /PDM_CLK: track 101.6 -> 43.4 mm, vias 1 -> 0
- net /FF_D: track 86.6 -> 31.0 mm, vias 2 -> 0
- net /I2C_DATA: track 84.9 -> 33.8 mm, vias 2 -> 0
- net /FF_Q: track 85.5 -> 34.7 mm, vias 2 -> 0
- net /FF_CLK: track 79.5 -> 31.1 mm, vias 1 -> 0
- net /DEC_CAP: track 40.1 -> 0.00 mm, vias 2 -> 0
- net /UART_TX: track 97.4 -> 62.0 mm
- net /SENSE_3_3V: track 55.8 -> 23.1 mm
- net Net-(J3-Pad8): track 29.2 -> 0.00 mm, vias 1 -> 0
- net GND: track 161.0 -> 132.2 mm, vias 15 -> 11
- net /BUTTON: track 28.3 -> 0.00 mm, vias 1 -> 0
- net unconnected-(U1-GP27-Pad32): track 0.00 -> 27.4 mm, vias 0 -> 2
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Other:
- board text added: "Dictofun-Fixture 1.4"
- board text removed: "Dictofun-Fixture 1.3"
